File: control-pcb/control-pcb/control-pcb.kicad_sch (KiCad schematic)
At the start: 22 parts, among them J1 Screw_Terminal_01x02, J2 Screw_Terminal_01x02, J3 Conn_01x03_Socket, J4 Conn_01x20_Pin, J6 Conn_01x15_Pin, J7 Conn_01x12_Pin, J8 Conn_01x06_Pin, J9 Conn_01x13_Pin, Q1 IRF540N, U1 ESP32-DEVKIT-V1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

Commit message: Modified schematic
Other:
- note added: "AC RECTIFICATION AND REGULATION"
- note added: "CURRENT SENSOR"
- note added: "MICROCONTROLLERS"
- note added: "POWER CONTROL CIRCUITRY"
- moved on the sheet: A1, J2, J4, J6, J7, J8, J9, Q1, R1, R2, U1, U2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
